File: PCB/V1.0/DMX-Card.brd (EAGLE design)
At the start: 48.3 x 24.1 mm, 34 parts, among them IC1 MAX481CSA, Q1 DMP3099L, X2 (NC3/NC5)FAH

Commit message: Update BOM
Parts:
- renumbered X2 to X1/2
Changed lines of the file:
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@@
 <attribute name="VALUE" x="25.78" y="18.885" size="1.016" layer="27" rot="R90"/>
 </element>
-<element name="X2" library="con-neutrik_ag" package="NC3FAH-NC5FAH-NOSILK" value="(NC3/NC5)FAH" x="33.02" y="12.065" smashed="yes" rot="R270">
+<element name="X1/2" library="con-neutrik_ag" package="NC3FAH-NC5FAH-NOSILK" value="(NC3/NC5)FAH" x="33.02" y="12.065" smashed="yes" rot="R270">
 <attribute name="VALUE" x="29.845" y="-0.635" size="1.27" layer="27" rot="R270" align="top-right"/>
 </element>
@@
 <contactref element="R12" pad="2"/>
 <contactref element="D6" pad="1"/>
-<contactref element="X2" pad="NC5-2"/>
-<contactref element="X2" pad="NC3-2"/>
+<contactref element="X1/2" pad="NC5-2"/>
+<contactref element="X1/2" pad="NC3-2"/>
 <wire x1="24.765" y1="16.51" x2="23.495" y2="16.51" width="0.508" layer="1"/>
 <wire x1="23.495" y1="16.51" x2="23.495" y2="16.725" width="0.508" layer="1"/>
@@
 <via x="27.94" y="17.78" extent="1-16" drill="0.6"/>
 <via x="25.4" y="17.78" extent="1-16" drill="0.6"/>
-<contactref element="X2" pad="NC5-1"/>
-<contactref element="X2" pad="NC3-1"/>
+<contactref element="X1/2" pad="NC5-1"/>
+<contactref element="X1/2" pad="NC3-1"/>
 <via x="25.4" y="3.175" extent="1-16" drill="0.6"/>
 <via x="34.29" y="1.27" extent="1-16" drill="0.6"/>
@@
 <wire x1="27.62" y1="14.775" x2="27.62" y2="15.555" width="0.508" layer="1"/>
 <wire x1="27.62" y1="15.555" x2="27.94" y2="15.875" width="0.508" layer="1"/>
-<contactref element="X2" pad="NC3-3"/>
+<contactref element="X1/2" pad="NC3-3"/>
 <wire x1="33.02" y1="12.065" x2="34.925" y2="10.16" width="0.508" layer="1"/>
 <wire x1="34.925" y1="10.16" x2="38.735" y2="10.16" width="0.508" layer="1"/>
